File: icarus schematic.kicad_sch (KiCad schematic)
At the start: 54 parts, among them J1 Conn_01x02_Socket, J2 USB_C_Receptacle_USB2.0_16P, J3 Conn_01x02_Socket, J4 Conn_01x02_Socket, J5 Conn_01x02_Socket, Q1 AO3400A, Q2 AO3400A, Q3 AO3400A, Q4 AO3400A, SW1 SW_Push(BOOt), SW2 SW_Push(EN), U2 BMI088, U3 AMS1117-3.3, U4 ESP32-S3-WROOM-1

Commit message: Add files via upload
Parts:
- C8: footprint Capacitor_SMD:C_0603_1608Metric_Pad1.08x0.95mm_HandSolder -> Capacitor_THT:C_Radial_D6.3mm_H5.0mm_P2.50mm
Connections:
- net GND: now also Q1.2 (S), Q2.2 (S), Q3.2 (S), Q4.2 (S)
- net M1: now also R8.1
- net M2: now also R9.1
- net M3: now also R10.1
- net M4: now also R11.1

Commit message: Add files via upload
Connections:
- net BOOT: no longer SW1.1
- net EN: no longer SW2.1
- net GND: now also SW1.1, SW2.1
Other:
- moved on the sheet: C2, C4

Commit message: Add files via upload
New updated mk 8 pcb and schematic
Parts:
- removed C8: 470uF, Capacitor_THT:C_Radial_D6.3mm_H5.0mm_P2.50mm, symbol Device:C
- added J6: Conn_01x02_Socket, Connector_JST:JST_EH_B2B-EH-A_1x02_P2.50mm_Vertical, symbol Connector:Conn_01x02_Socket
- added J8: Conn_01x02_Pin, Connector_JST:JST_SH_SM02B-SRSS-TB_1x02-1MP_P1.00mm_Horizontal, symbol Connector:Conn_01x02_Pin
- TP5, TP6: footprint TestPoint:TestPoint_Pad_4.0x4.0mm -> TestPoint:TestPoint_THTPad_2.0x2.0mm_Drill1.0mm
Connections:
- net 5V: now also C10.1, C11.1, C12.1, C13.1, D2.1 (K), D3.1 (K), D4.1 (K), D5.1 (K), J1.2 (Pin_2), J3.2 (Pin_2), J4.2 (Pin_2), J5.2 (Pin_2), TP5.1, J6.1 (Pin_1), J8.2 (Pin_2)
- net GND: now also J6.2 (Pin_2), J8.1 (Pin_1)
Other:
- note added: "Camera socket"
- moved on the sheet: C2, C4, C5, C6, C9, R12, R2, R3, R4, R5, R6, R7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

Commit message: Add files via upload
corrected final mk 8
Connections:
- net SD02 is gone; now on net SD01: U2.10 (SDO2), U4.22 (IO14)
Changed lines of the file:
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@@
+	)
+	(junction
+		(at 165.1 38.1)
+		(diameter 0)
+		(color 0 0 0 0)
 	)
 	(junction
@@
 	)
 	(junction
+		(at 76.2 116.84)
+		(diameter 0)
+		(color 0 0 0 0)
+	)
+	(junction
 		(at 153.67 50.8)
 		(diameter 0)
@@
 	(wire
 		(pts
+			(xy 76.2 116.84) (xy 77.47 116.84)
+		)
+		(stroke
+			(width 0)
+			(type default)
+		)
+	)
+	(wire
+		(pts
 			(xy 40.64 111.76) (xy 44.45 111.76)
 		)
@@
 	(wire
 		(pts
-			(xy 74.93 116.84) (xy 77.47 116.84)
+			(xy 74.93 116.84) (xy 76.2 116.84)
 		)
 		(stroke
@@
 	(wire
 		(pts
-			(xy 166.37 38.1) (xy 163.83 38.1)
+			(xy 166.37 38.1) (xy 165.1 38.1)
 		)
 		(stroke
@@
 	(wire
 		(pts
-			(xy 74.93 119.38) (xy 77.47 119.38)
-		)
-		(stroke
-			(width 0)
-			(type default)
-		)
-	)
-	(wire
-		(pts
 			(xy 162.56 125.73) (xy 162.56 135.89)
 		)
@@
 	(wire
 		(pts
+			(xy 74.93 119.38) (xy 76.2 119.38)
+		)
+		(stroke
+			(width 0)
+			(type default)
+		)
+	)
+	(wire
+		(pts
 			(xy 39.37 36.83) (xy 27.94 36.83)
 		)
@@
 	(wire
 		(pts
+			(xy 76.2 119.38) (xy 76.2 116.84)
+		)
+		(stroke
+			(width 0)
+			(type default)
+		)
+	)
+	(wire
+		(pts
 			(xy 182.88 64.77) (xy 186.69 64.77)
 		)
@@
 	(wire
 		(pts
+			(xy 163.83 40.64) (xy 165.1 40.64)
+		)
+		(stroke
+			(width 0)
+			(type default)
+		)
+	)
+	(wire
+		(pts
 			(xy 173.99 17.78) (xy 173.99 30.48)
 		)
@@
 	(wire
 		(pts
+			(xy 165.1 40.64) (xy 165.1 38.1)
+		)
+		(stroke
+			(width 0)
+			(type default)
+		)
+	)
+	(wire
+		(pts
 			(xy 125.73 72.39) (xy 134.62 72.39)
 		)
@@
 	(wire
 		(pts
+			(xy 165.1 38.1) (xy 163.83 38.1)
+		)
+		(stroke
+			(width 0)
+			(type default)
+		)
+	)
+	(wire
+		(pts
 			(xy 170.18 93.98) (xy 170.18 106.68)
 		)
@@
 	(wire
 		(pts
-			(xy 163.83 40.64) (xy 166.37 40.64)
-		)
-		(stroke
-			(width 0)
-			(type default)
-		)
-	)
-	(wire
-		(pts
 			(xy 256.54 34.29) (xy 259.08 34.29)
 		)
@@
 			(width 0)
 			(type default)
-		)
-	)
-	(label "SD02"
-		(at 77.47 119.38 0)
-		(effects
-			(font
-				(size 1.27 1.27)
-			)
-			(justify left bottom)
 		)
 	)
@@
 		)
 	)
-	(label "SD02"
-		(at 166.37 40.64 0)
-		(effects
-			(font
-				(size 1.27 1.27)
-			)
-			(justify left bottom)
-		)
-	)

Commit message: Add files via upload
final final pcb mk 8
Connections:
- net INT1: no longer names the net of U4.4 (IO4)
- net INT1: no longer U2.16 (INT1)
- net INT3: no longer names the net of U4.5 (IO5)
- net INT3: no longer U2.12 (INT3)
- no-connect marks 25 -> 29
Changed lines of the file:
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@@
+	)
+	(no_connect
+		(at 74.93 96.52)
 	)
 	(no_connect
@@
 	)
 	(no_connect
+		(at 74.93 93.98)
+	)
+	(no_connect
 		(at 44.45 93.98)
 	)
@@
 	)
 	(no_connect
+		(at 138.43 38.1)
+	)
+	(no_connect
 		(at 243.84 49.53)
 	)
@@
 	)
 	(no_connect
+		(at 138.43 27.94)
+	)
+	(no_connect
 		(at 74.93 86.36)
 	)
@@
 	(wire
 		(pts
-			(xy 74.93 96.52) (xy 77.47 96.52)
-		)
-		(stroke
-			(width 0)
-			(type default)
-		)
-	)
-	(wire
-		(pts
 			(xy 119.38 72.39) (xy 119.38 81.28)
 		)
@@
 		(pts
 			(xy 128.27 16.51) (xy 128.27 30.48)
-		)
-		(stroke
-			(width 0)
-			(type default)
-		)
-	)
-	(wire
-		(pts
-			(xy 74.93 93.98) (xy 77.47 93.98)
 		)
 		(stroke
@@
 		)
 	)
-	(label "INT3"
-		(at 77.47 96.52 0)
-		(effects
-			(font
-				(size 1.27 1.27)
-			)
-			(justify left bottom)
-		)
-	)
 	(label "3.3V"
 		(at 85.09 17.78 0)
@@
 		)
 	)
-	(label "INT1"
-		(at 138.43 27.94 180)
-		(effects
-			(font
-				(size 1.27 1.27)
-			)
-			(justify right bottom)
-		)
-	)
 	(label "EN"
 		(at 105.41 27.94 0)
@@
 		)
 	)
-	(label "INT3"
-		(at 138.43 38.1 180)
-		(effects
-			(font
-				(size 1.27 1.27)
-			)
-			(justify right bottom)
-		)
-	)
 	(label "SCK"
 		(at 77.47 114.3 0)
@@
 		(effects
 			(font
-				(size 1.27 1.27)
-			)
-			(justify left bottom)
-		)
-	)
-	(label "INT1"
-		(at 77.47 93.98 0)
-		(effects
-			(font
