File: icarus schematic.kicad_pcb (KiCad board)
At the start: 2 copper layers, 40 x 60 mm, 54 parts, among them J1 Conn_01x02_Socket, J2 USB_C_Receptacle_USB2.0_16P, J3 Conn_01x02_Socket, J4 Conn_01x02_Socket, J5 Conn_01x02_Socket, Q1 AO3400A, Q2 AO3400A, Q3 AO3400A, Q4 AO3400A, SW1 SW_Push(BOOt), SW2 SW_Push(EN), U2 BMI088, U3 AMS1117-3.3, U4 ESP32-S3-WROOM-1

Commit message: Add files via upload
Icarus pcb mk 3 structure is right but the schematic is wrong
Parts:
- moved TP4 48.4 mm to (165.4, 101.6), turned to 180 degrees
- moved R11 47.0 mm to (165.3, 97.7), turned to 90 degrees
- moved C11 40.0 mm to (160.5, 92.6), turned to 90 degrees
- moved C10 39.8 mm to (135.6, 92.8), turned to 90 degrees
- moved TP3 38.3 mm to (164.5, 122.8), turned to 180 degrees
- moved Q1 36.5 mm to (130.8, 92.8)
- moved Q4 36.4 mm to (165.2, 93.1)
- moved J1 36.3 mm to (131.6, 86.5), turned to 0 degrees
- moved J5 36.2 mm to (161.4, 86.2), turned to 0 degrees
- moved D4 35.4 mm to (159.4, 127.3)
- moved TP2 34.8 mm to (130.8, 101.4), turned to 180 degrees
- moved R10 32.9 mm to (164.7, 127.4), turned to 90 degrees
- moved R6 31.7 mm to (155.6, 116.2), turned to 0 degrees
- moved SW1 28.9 mm to (142.4, 122.4), turned to -90 degrees
- moved D5 27.3 mm to (160.6, 97.7)
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
Commit message: Add files via upload
Parts:
- added R10: 10k, Resistor_SMD:R_0603_1608Metric_Pad0.98x0.95mm_HandSolder, F.Cu at (159.4, 122.8)
- added R11: 10k, Resistor_SMD:R_0603_1608Metric_Pad0.98x0.95mm_HandSolder, F.Cu at (160.8, 101.7)
- added R8: 10k, Resistor_SMD:R_0603_1608Metric_Pad0.98x0.95mm_HandSolder, F.Cu at (135.5, 101.4)
- added R9: 10k, Resistor_SMD:R_0603_1608Metric_Pad0.98x0.95mm_HandSolder, F.Cu at (136.1, 123.1)
Connections:
- Q1 pad 2: Net-(Q1-S) -> GND
- Q2 pad 2: Net-(Q2-S) -> GND
- Q3 pad 2: Net-(Q3-S) -> GND
- Q4 pad 2: Net-(Q4-S) -> GND

Commit message: Add files via upload
mk 4 with the routing
Parts:
- moved R4 16.1 mm to (140.1, 105.6), turned to 180 degrees
- moved TP1 7.03 mm to (137.8, 123.0), turned to 0 degrees
- moved TP4 5.64 mm to (159.8, 101.6), turned to 0 degrees
- moved R9 5.34 mm to (130.7, 122.9)
- moved R10 5.23 mm to (164.6, 122.8)
- moved R11 4.41 mm to (165.2, 101.5), turned to 180 degrees
- moved TP3 4.14 mm to (160.4, 122.7), turned to 0 degrees
- moved TP2 4.09 mm to (134.8, 101.3), turned to 0 degrees
- moved R8 3.95 mm to (131.6, 101.3), turned to 180 degrees
- moved R7 3.26 mm to (158.7, 105.3)
- moved R13 3.08 mm to (149.0, 129.5), turned to 90 degrees
- moved R5 2.92 mm to (156.7, 110.3), turned to -90 degrees
- moved C9 2.63 mm to (138.1, 109.8), turned to 90 degrees
- moved R12 2.61 mm to (140.6, 109.2)
- moved R9 1.79 mm to (132.6, 127.4), turned to 180 degrees
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Routing:
- net GND: track 0.00 -> 228.0 mm, vias 0 -> 14
- net Net-(D2-K): track 0.00 -> 136.5 mm, vias 0 -> 4
- net /3.3V: track 0.00 -> 79.4 mm, vias 0 -> 6
- net /EN: track 0.00 -> 56.0 mm, vias 0 -> 4
- net /USB_D+: track 0.00 -> 53.4 mm, vias 0 -> 4
- net /USB_D-: track 0.00 -> 51.2 mm, vias 0 -> 2
- net /INT1: track 0.00 -> 48.5 mm, vias 0 -> 2
- net /M2: track 0.00 -> 45.6 mm, vias 0 -> 4
- net /BOOT: track 0.00 -> 38.3 mm, vias 0 -> 2
- net /INT3: track 0.00 -> 30.7 mm, vias 0 -> 2
- net /5V: track 0.00 -> 30.1 mm, vias 0 -> 2
- net Net-(D3-A): track 0.00 -> 27.6 mm, vias 0 -> 2
- net Net-(D4-A): track 0.00 -> 26.1 mm, vias 0 -> 2
- net /M3: track 0.00 -> 23.3 mm, vias 0 -> 2
- net Net-(U4-IO40): track 0.00 -> 23.2 mm, vias 0 -> 2
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
Commit message: Add files via upload
Parts:
- removed C8: 470uF, Capacitor_SMD:C_0603_1608Metric_Pad1.08x0.95mm_HandSolder
- moved Q4 53.1 mm to (129.4, 132.3), turned to 0 degrees
- moved J5 50.4 mm to (133.7, 128.2), turned to 180 degrees
- moved TP5 50.1 mm to (122.0, 135.1)
- moved TP6 49.3 mm to (122.0, 140.2)
- moved C11 48.7 mm to (132.3, 132.2), turned to 90 degrees
- moved D7 48.5 mm to (110.0, 111.9)
- moved R11 47.8 mm to (126.4, 129.4), turned to 0 degrees
- moved SW2 46.9 mm to (109.7, 106.3), turned to 90 degrees
- moved J1 46.3 mm to (110.3, 127.6)
- moved C10 46.0 mm to (111.8, 132.1), turned to 90 degrees
- moved R11 45.9 mm to (135.0, 133.0), turned to 0 degrees
- moved TP4 45.5 mm to (126.2, 132.3)
- moved C4 45.4 mm to (109.5, 102.8), turned to 180 degrees
- moved D2 44.2 mm to (109.0, 133.0)
- moved R3 43.8 mm to (109.6, 101.4), turned to 0 degrees
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Routing:
- net GND: track 228.0 -> 0.00 mm, vias 14 -> 0
- net Net-(D2-K): track 136.5 -> 0.00 mm, vias 4 -> 0
- net /3.3V: track 79.4 -> 0.00 mm, vias 6 -> 0
- net /EN: track 56.0 -> 0.00 mm, vias 4 -> 0
- net /USB_D+: track 53.4 -> 0.00 mm, vias 4 -> 0
- net /USB_D-: track 51.2 -> 0.00 mm, vias 2 -> 0
- net /INT1: track 48.5 -> 0.00 mm, vias 2 -> 0
- net /M2: track 45.6 -> 0.00 mm, vias 4 -> 0
- net /BOOT: track 38.3 -> 0.00 mm, vias 2 -> 0
- net /INT3: track 30.7 -> 0.00 mm, vias 2 -> 0
- net /5V: track 30.1 -> 0.00 mm, vias 2 -> 0
- net Net-(D3-A): track 27.6 -> 0.00 mm, vias 2 -> 0
- net Net-(D4-A): track 26.1 -> 0.00 mm, vias 2 -> 0
- net /M3: track 23.3 -> 0.00 mm, vias 2 -> 0
- net Net-(U4-IO40): track 23.2 -> 0.00 mm, vias 2 -> 0
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- added copper zone on B.Cu, net GND
- added copper zone on F.Cu, net GND
Other:
- board size 40 x 60 mm -> 30 x 50 mm

Commit message: Add files via upload
Parts:
- removed the R10 at (135.8, 136.0)
- removed the R11 at (135.0, 133.0)
- removed the R8 at (108.9, 131.2)
- removed the R9 at (108.9, 135.4)
- moved C1 35.9 mm to (101.2, 142.6), turned to 180 degrees
- moved U3 35.2 mm to (103.0, 137.3), turned to -90 degrees
- moved C7 35.0 mm to (104.9, 142.6), turned to 0 degrees
- moved D6 32.9 mm to (90.2, 110.8), turned to 90 degrees
- moved C3 29.0 mm to (100.7, 131.9), turned to 0 degrees
- moved R1 28.5 mm to (100.6, 130.4)
- moved D1 28.2 mm to (104.8, 131.4)
- moved Q2 23.7 mm to (94.0, 136.6)
- moved TP6 23.6 mm to (115.3, 117.5)
- moved D3 23.6 mm to (89.1, 136.8), turned to -90 degrees
- moved C2 23.2 mm to (111.0, 115.5), turned to 180 degrees
- moved R2 22.7 mm to (111.6, 117.3), turned to 90 degrees
- moved C10 21.7 mm to (90.0, 131.8), turned to 0 degrees
- moved J5 21.5 mm to (112.2, 127.5), turned to 0 degrees
- moved R8 20.8 mm to (97.0, 132.4), turned to -90 degrees
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Connections:
- SW1 pad 1: /BOOT -> GND
- SW2 pad 1: /EN -> GND

Commit message: Icarus PCB mk7 **finalised**
Parts:
- moved J5 50.1 mm to (161.7, 119.2), turned to -90 degrees
- moved J3 49.9 mm to (161.1, 130.8), turned to 90 degrees
- moved D2 49.5 mm to (138.3, 122.7), turned to 90 degrees
- moved C6 49.4 mm to (149.7, 113.2)
- moved D3 49.4 mm to (137.5, 126.6), turned to 0 degrees
- moved TP3 47.8 mm to (153.2, 126.4), turned to 90 degrees
- moved R7 47.6 mm to (161.6, 87.8)
- moved R6 47.6 mm to (161.6, 90.3)
- moved R5 47.6 mm to (161.5, 92.7)
- moved R4 47.5 mm to (161.5, 95.1)
- moved C10 47.4 mm to (136.6, 122.7), turned to 90 degrees
- moved C13 47.2 mm to (137.5, 128.8), turned to 0 degrees
- moved U4 47.1 mm to (149.1, 91.3)
- moved TP6 47.0 mm to (161.4, 108.3)
- moved TP5 47.0 mm to (161.4, 113.4)
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Routing:
- net /3.3V: track 0.00 -> 82.8 mm, vias 0 -> 3
- net /M2: track 0.00 -> 51.5 mm, vias 0 -> 2
- net /M3: track 0.00 -> 50.5 mm, vias 0 -> 2
- net /M4: track 0.00 -> 42.4 mm, vias 0 -> 2
- net /M1: track 0.00 -> 40.5 mm, vias 0 -> 2
- net /INT1: track 0.00 -> 32.3 mm, vias 0 -> 2
- net Net-(D2-K): track 0.00 -> 29.1 mm, vias 0 -> 2
- net /INT3: track 0.00 -> 26.0 mm, vias 0 -> 2
- net Net-(D6-A): track 0.00 -> 22.7 mm, vias 0 -> 2
- net /USB_D-: track 0.00 -> 18.0 mm, vias 0 -> 2
- net /USB_D+: track 0.00 -> 17.7 mm, vias 0 -> 3
- net /CSB2: track 0.00 -> 16.4 mm
- net /5V: track 0.00 -> 15.7 mm
- net GND: track 0.00 -> 14.0 mm, vias 0 -> 7
- net /SCK: track 0.00 -> 10.8 mm, vias 0 -> 2
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- added copper zone on F.Cu, net /3.3V
- added copper zone on F.Cu, net /EN
- added copper zone on F.Cu, net Net-(D1-A)
- added copper zone on F.Cu, net Net-(D2-A)
- added copper zone on F.Cu, net Net-(D2-K)
- added copper zone on F.Cu, net Net-(D3-A)
- added copper zone on F.Cu, net Net-(D4-A)
- added copper zone on F.Cu, net Net-(D5-A)
Other:
- board size 30 x 50 mm -> 35 x 50 mm

Commit message: Add files via upload
New updated mk 8 pcb and schematic
Parts:
- added J6: Conn_01x02_Socket, Connector_JST:JST_EH_B2B-EH-A_1x02_P2.50mm_Vertical, F.Cu at (161.1, 112.7)
- added J8: Conn_01x02_Pin, Connector_JST:JST_SH_SM02B-SRSS-TB_1x02-1MP_P1.00mm_Horizontal, F.Cu at (132.5, 113.2)
- TP5, TP6: footprint TestPoint:TestPoint_Pad_4.0x4.0mm -> TestPoint:TestPoint_THTPad_2.0x2.0mm_Drill1.0mm
- moved D6 11.7 mm to (144.6, 117.8)
- moved D7 6.40 mm to (138.2, 110.0), turned to 180 degrees
- moved R14 5.00 mm to (131.8, 108.7)
- moved TP6 4.26 mm to (157.5, 110.0)
- moved TP5 3.93 mm to (157.5, 113.0)
- moved R8 0.76 mm to (140.0, 118.6)
- moved R11 0.37 mm to (153.6, 118.5)
- moved U4 0.14 mm to (149.1, 91.4)
- moved J2 0.14 mm to (133.1, 102.5)
Connections:
- C10 pad 1: Net-(D2-K) -> /5V
- C11 pad 1: Net-(D2-K) -> /5V
- C12 pad 1: Net-(D2-K) -> /5V
- C13 pad 1: Net-(D2-K) -> /5V
- D2 pad 1: Net-(D2-K) -> /5V
- D3 pad 1: Net-(D2-K) -> /5V
- D4 pad 1: Net-(D2-K) -> /5V
- D5 pad 1: Net-(D2-K) -> /5V
- J1 pad 2: Net-(D2-K) -> /5V
- J3 pad 2: Net-(D2-K) -> /5V
- J4 pad 2: Net-(D2-K) -> /5V
- J5 pad 2: Net-(D2-K) -> /5V
- TP5 pad 1: Net-(D2-K) -> /5V
Routing:
- net /5V: track 15.7 -> 57.2 mm, vias 0 -> 2
- net Net-(D2-K): track 29.1 -> 0.00 mm, vias 2 -> 0
- net Net-(D6-A): track 22.7 -> 28.6 mm
- net Net-(J2-CC2): track 5.83 -> 9.99 mm
- net /3.3V: track 82.8 -> 80.1 mm
- net /M1: track 40.5 -> 38.0 mm
- net GND: track 14.0 -> 16.3 mm, vias 7 -> 9
- net /SCK: track 10.8 -> 9.95 mm
- net /M4: track 42.4 -> 41.7 mm
- net /USB_D-: track 18.0 -> 18.7 mm
- net /INT3: track 26.0 -> 25.4 mm
- added copper zone on F.Cu, net /5V
- removed copper zone on F.Cu, net Net-(D2-K)

Commit message: Add files via upload
corrected final mk 8
Connections:
- U2 pad 10: /SD02 -> /SD01
- U4 pad 22: /SD02 -> /SD01
Routing:
- net /SD02: track 9.15 -> 0.00 mm, vias 2 -> 0
- net /SD01: track 5.26 -> 9.30 mm, vias 0 -> 2
Changed lines of the file:
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@@
 			(size 1.5 0.9)
 			(layers "F.Cu" "F.Mask" "F.Paste")
-			(net "/SD02")
+			(net "/SD01")
 			(pinfunction "IO14_22")
 			(pintype "bidirectional")
@@
 			(layers "F.Cu" "F.Mask" "F.Paste")
 			(roundrect_rratio 0.25)
-			(net "/SD02")
+			(net "/SD01")
 			(pinfunction "SDO2_10")
 			(pintype "output")
@@
 		)
 		(property "Value" "USB_C_Receptacle_USB2.0_16P"
-			(at 1.075 5 270)
+			(at 0.07 4.68 270)
 			(unlocked yes)
 			(layer "F.Fab")
@@
 	)
 	(segment
-		(start 147.39 105.49)
-		(end 147.39 103.955)
+		(start 146.949265 105.930735)
+		(end 147.39 105.49)
 		(width 0.2)
 		(layer "F.Cu")
@@
 	)
 	(segment
-		(start 147.39 103.955)
-		(end 147.195 103.76)
+		(start 144.37 107.22)
+		(end 144.37 107.665)
 		(width 0.2)
 		(layer "F.Cu")
@@
 	)
 	(segment
-		(start 144.37 107.22)
-		(end 144.37 107.665)
+		(start 147.39 105.49)
+		(end 147.39 103.955)
 		(width 0.2)
 		(layer "F.Cu")
@@
 	)
 	(segment
-		(start 146.949265 105.930735)
-		(end 147.39 105.49)
+		(start 147.39 103.955)
+		(end 147.195 103.76)
 		(width 0.2)
 		(layer "F.Cu")
@@
 	)
 	(segment
-		(start 149.735 103.76)
-		(end 149.735 105.445)
+		(start 145.307847 107.309653)
+		(end 145.307847 107.747847)
 		(width 0.2)
 		(layer "F.Cu")
@@
 	)
 	(segment
-		(start 148.0125 107.1675)
-		(end 148.0125 108.3075)
+		(start 149.735 105.015)
+		(end 148.0125 106.7375)
 		(width 0.2)
 		(layer "F.Cu")
@@
 	)
 	(segment
-		(start 149.735 105.445)
-		(end 148.0125 107.1675)
+		(start 149.735 103.9)
+		(end 149.735 105.015)
 		(width 0.2)
 		(layer "F.Cu")
@@
 	)
 	(segment
-		(start 145.307847 107.309653)
-		(end 145.307847 107.747847)
+		(start 148.0125 106.8)
+		(end 148.0125 108.3075)
 		(width 0.2)
 		(layer "F.Cu")
-		(net "/SD02")
+		(net "/SD01")
 	)
 	(segment
-		(start 151.005 105.035)
-		(end 151.005 103.76)
+		(start 145.401597 107.215903)
+		(end 145.307847 107.309653)
 		(width 0.2)
 		(layer "F.Cu")
-		(net "/SD02")
+		(net "/SD01")
 	)
 	(segment
-		(start 145.401597 107.215903)
-		(end 145.307847 107.309653)
+		(start 148.0125 106.7375)
+		(end 148.0125 106.8)
 		(width 0.2)
 		(layer "F.Cu")
-		(net "/SD02")
+		(net "/SD01")
 	)
 	(segment
@@
 		(width 0.2)
 		(layer "F.Cu")
-		(net "/SD02")
+		(net "/SD01")
 	)
 	(segment
@@
 		(width 0.2)
 		(layer "F.Cu")
-		(net "/SD02")
-	)
-	(segment
-		(start 149.67 106.37)
-		(end 151.005 105.035)
-		(width 0.2)
-		(layer "F.Cu")
-		(net "/SD02")
+		(net "/SD01")
 	)
 	(via
-		(at 149.67 106.37)
+		(at 148.0125 106.8)
 		(size 0.6)
 		(drill 0.3)
 		(layers "F.Cu" "B.Cu")
-		(net "/SD02")
+		(net "/SD01")
 	)
 	(via
@@
 		(drill 0.3)
 		(layers "F.Cu" "B.Cu")
-		(net "/SD02")
+		(net "/SD01")
 	)
 	(segment
-		(start 149.13 106.91)
-		(end 149.67 106.37)
+		(start 145.91 106.76)
+		(end 147.9725 106.76)
 		(width 0.2)
 		(layer "B.Cu")
-		(net "/SD02")
+		(net "/SD01")
 	)
 	(segment
-		(start 145.76 106.91)
-		(end 149.13 106.91)
+		(start 145.401597 107.215903)
+		(end 145.454097 107.215903)
 		(width 0.2)
 		(layer "B.Cu")
-		(net "/SD02")
+		(net "/SD01")
 	)
 	(segment
@@
 		(width 0.2)
 		(layer "B.Cu")
-		(net "/SD02")
+		(net "/SD01")
 	)
 	(segment
-		(start 145.454097 107.215903)
-		(end 145.76 106.91)
+		(start 147.9725 106.76)
+		(end 148.0125 106.8)
 		(width 0.2)
 		(layer "B.Cu")
-		(net "/SD02")
+		(net "/SD01")
 	)
 	(segment
@@
 		(width 0.2)
 		(layer "B.Cu")
-		(net "/SD02")
+		(net "/SD01")
 	)
 	(segment
-		(start 145.401597 107.215903)
-		(end 145.454097 107.215903)
+		(start 145.454097 107.215903)
+		(end 145.91 106.76)
 		(width 0.2)
 		(layer "B.Cu")
-		(net "/SD02")
+		(net "/SD01")
 	)
 	(segment
