File: icarus schematic.kicad_pcb (KiCad board)
At the start: 2 copper layers, 35 x 50 mm, 55 parts, among them J1 Conn_01x02_Socket, J2 USB_C_Receptacle_USB2.0_16P, J3 Conn_01x02_Socket, J4 Conn_01x02_Socket, J5 Conn_01x02_Socket, J6 Conn_01x02_Socket, J8 Conn_01x02_Pin, Q1 AO3400A, Q2 AO3400A, Q3 AO3400A, Q4 AO3400A, SW1 SW_Push(BOOt), SW2 SW_Push(EN), U2 BMI088, U3 AMS1117-3.3, U4 ESP32-S3-WROOM-1

Commit message: Add files via upload
final final pcb mk 8
Parts:
- moved J8 0.25 mm to (132.5, 113.0)
- moved J1 0.13 mm to (132.7, 119.3)
- moved J4 0.12 mm to (132.1, 130.8)
Connections:
- U2 pad 12: /INT3 -> unconnected-(U2-INT3-Pad12)
- U2 pad 16: /INT1 -> unconnected-(U2-INT1-Pad16)
- U4 pad 4: /INT1 -> unconnected-(U4-IO4-Pad4)
- U4 pad 5: /INT3 -> unconnected-(U4-IO5-Pad5)
Routing:
- net /INT1: track 32.0 -> 0.00 mm, vias 2 -> 0
- net /INT3: track 25.4 -> 0.00 mm, vias 2 -> 0
- net /3.3V: track 80.1 -> 77.4 mm
- net /CSB2: track 16.4 -> 14.7 mm
- net /SD01: track 9.30 -> 10.7 mm

Commit message: New PCB mk8
Parts:
- added G***: LOGO, LOGO, B.Cu at (147.4, 129.8)
Other:
- board text added: "ICARUS"
