File: schematic/icarus schematic.kicad_sch (KiCad schematic)
At the start: 54 parts, among them J1 Conn_01x02_Socket, J2 USB_C_Receptacle_USB2.0_16P, J3 Conn_01x02_Socket, J4 Conn_01x02_Socket, J5 Conn_01x02_Socket, Q1 AO3400A, Q2 AO3400A, Q3 AO3400A, Q4 AO3400A, SW1 SW_Push(BOOt), SW2 SW_Push(EN), U2 BMI088, U3 AMS1117-3.3, U4 ESP32-S3-WROOM-1

Commit message: Changes to the schematic
Connections:
- net SD02 is gone; now on net SD01: U2.10 (SDO2), U4.22 (IO14)
Changed lines of the file:
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@@
+	)
+	(junction
+		(at 86.36 26.67)
+		(diameter 0)
+		(color 0 0 0 0)
 	)
 	(junction
@@
 	)
 	(junction
-		(at 86.36 27.94)
-		(diameter 0)
-		(color 0 0 0 0)
-	)
-	(junction
 		(at 279.4 21.59)
 		(diameter 0)
@@
 	)
 	(junction
+		(at 77.47 113.03)
+		(diameter 0)
+		(color 0 0 0 0)
+	)
+	(junction
 		(at 156.21 50.8)
 		(diameter 0)
@@
 	)
 	(junction
+		(at 168.91 38.1)
+		(diameter 0)
+		(color 0 0 0 0)
+	)
+	(junction
 		(at 119.38 106.68)
 		(diameter 0)
@@
 	(wire
 		(pts
+			(xy 86.36 26.67) (xy 86.36 35.56)
+		)
+		(stroke
+			(width 0)
+			(type default)
+		)
+	)
+	(wire
+		(pts
 			(xy 49.53 33.02) (xy 49.53 36.83)
 		)
@@
 	(wire
 		(pts
-			(xy 74.93 27.94) (xy 74.93 26.67)
-		)
-		(stroke
-			(width 0)
-			(type default)
-		)
-	)
-	(wire
-		(pts
 			(xy 74.93 113.03) (xy 77.47 113.03)
 		)
@@
 	(wire
 		(pts
-			(xy 168.91 38.1) (xy 166.37 38.1)
-		)
-		(stroke
-			(width 0)
-			(type default)
-		)
-	)
-	(wire
-		(pts
 			(xy 186.69 72.39) (xy 194.31 72.39)
 		)
@@
 	(wire
 		(pts
-			(xy 74.93 27.94) (xy 86.36 27.94)
+			(xy 74.93 26.67) (xy 86.36 26.67)
 		)
 		(stroke
@@
 	(wire
 		(pts
-			(xy 86.36 27.94) (xy 86.36 35.56)
-		)
-		(stroke
-			(width 0)
-			(type default)
-		)
-	)
-	(wire
-		(pts
 			(xy 170.18 115.57) (xy 173.99 115.57)
 		)
@@
 	(wire
 		(pts
+			(xy 77.47 113.03) (xy 77.47 115.57)
+		)
+		(stroke
+			(width 0)
+			(type default)
+		)
+	)
+	(wire
+		(pts
 			(xy 170.18 64.77) (xy 175.26 64.77)
 		)
@@
 	(wire
 		(pts
-			(xy 86.36 25.4) (xy 86.36 27.94)
+			(xy 86.36 25.4) (xy 86.36 26.67)
 		)
 		(stroke
@@
 	(wire
 		(pts
+			(xy 168.91 38.1) (xy 170.18 38.1)
+		)
+		(stroke
+			(width 0)
+			(type default)
+		)
+	)
+	(wire
+		(pts
 			(xy 139.7 116.84) (xy 144.78 116.84)
 		)
@@
 	(wire
 		(pts
+			(xy 77.47 113.03) (xy 80.01 113.03)
+		)
+		(stroke
+			(width 0)
+			(type default)
+		)
+	)
+	(wire
+		(pts
 			(xy 111.76 101.6) (xy 106.68 101.6)
 		)
@@
 	(wire
 		(pts
+			(xy 166.37 38.1) (xy 168.91 38.1)
+		)
+		(stroke
+			(width 0)
+			(type default)
+		)
+	)
+	(wire
+		(pts
 			(xy 151.13 50.8) (xy 156.21 50.8)
 		)
@@
 	(wire
 		(pts
+			(xy 168.91 38.1) (xy 168.91 40.64)
+		)
+		(stroke
+			(width 0)
+			(type default)
+		)
+	)
+	(wire
+		(pts
 			(xy 111.76 93.98) (xy 111.76 101.6)
 		)
@@
 			(width 0)
 			(type default)
-		)
-	)
-	(label "SD02"
-		(at 77.47 115.57 0)
-		(effects
-			(font
-				(size 1.27 1.27)
-			)
-			(justify left bottom)
 		)
 	)
@@
 	)
 	(label "SD01"
-		(at 168.91 38.1 0)
+		(at 80.01 113.03 0)
 		(effects
 			(font
@@
 		)
 	)
+	(label "SD01"
+		(at 170.18 38.1 0)
+		(effects
+			(font
+				(size 1.27 1.27)
+			)
+			(justify left bottom)
+		)
+	)
 	(label "M3"
 		(at 33.02 105.41 180)
@@
 		)
 	)
-	(label "SD01"
-		(at 77.47 113.03 0)
-		(effects
-			(font
-				(size 1.27 1.27)
-			)
-			(justify left bottom)
-		)
-	)
 	(label "SDI"
 		(at 77.47 107.95 0)
@@
 		)
 	)
-	(label "SD02"
-		(at 168.91 40.64 0)
-		(effects
-			(font
-				(size 1.27 1.27)
-			)
-			(justify left bottom)
-		)
-	)
 	(label "CSB1"
 		(at 166.37 27.94 0)
@@
 	)
 	(label "BOOT"
-		(at 86.36 27.94 0)
-		(effects
-			(font
+		(at 86.36 26.67 0)
+		(effects
+			(font
