File: Schematic and PCB/icarus.kicad_sch (KiCad schematic)
At the start: 55 parts, among them J1 Conn_01x02_Socket, J2 USB_C_Receptacle_USB2.0_16P, J3 Conn_01x02_Socket, J4 Conn_01x02_Socket, J5 Conn_01x02_Socket, J6 Conn_01x02_Socket, J8 Conn_01x02_Pin, Q1 AO3400A, Q2 AO3400A, Q3 AO3400A, Q4 AO3400A, SW1 SW_Push(BOOt), SW2 SW_Push(EN), U2 BMI088, U3 AMS1117-3.3, U4 ESP32-S3-WROOM-1

Commit message: FINAL PCB
Parts:
- removed D2, D3, D4, D5: 1N5819, Diode_SMD:D_0603_1608Metric_Pad1.05x0.95mm_HandSolder, symbol Diode:1N5819
- added D2, D3, D4, D5: SS24, Diode_SMD:D_SMA, symbol Diode:SS24
- C1, C3, C7: footprint Capacitor_SMD:C_0402_1005Metric_Pad0.74x0.62mm_HandSolder -> Capacitor_SMD:C_0805_2012Metric
- C10, C11, C12, C13: footprint Capacitor_SMD:C_0603_1608Metric_Pad1.08x0.95mm_HandSolder -> Capacitor_SMD:C_1206_3216Metric
- C2, C4, C5, C6, C9: footprint Capacitor_SMD:C_0402_1005Metric_Pad0.74x0.62mm_HandSolder -> Capacitor_SMD:C_0603_1608Metric
- R1, R12, R13, R14, R2, R3: footprint Resistor_SMD:R_0402_1005Metric_Pad0.72x0.64mm_HandSolder -> Resistor_SMD:R_0603_1608Metric
- R10, R11, R4, R5, R6, R7, R8, R9: footprint Resistor_SMD:R_0603_1608Metric_Pad0.98x0.95mm_HandSolder -> Resistor_SMD:R_0603_1608Metric
Connections:
- net 5V: now also D2.1 (K), D3.1 (K), D4.1 (K), D5.1 (K)
- net at C10.2, J1.1 (Pin_1), Q1.3 (D)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: now also D2.2 (A)
- net at C11.2, J5.1 (Pin_1), Q4.3 (D)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: now also D5.2 (A)
- net at C13.2, J4.1 (Pin_1), Q2.3 (D)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: now also D3.2 (A)
- net at C12.2, J3.1 (Pin_1), Q3.3 (D)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: now also D4.2 (A)
